File: hw/a2ext-carrier/a2ext-carrier.kicad_sch (KiCad schematic)
At the start: 30 parts, among them J1 Apple II slot, counter-clockw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, J2 Daughterboard IDC20, M1 WeAct RP2350B V1.0 (prepared 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, Q1 2N7002, U1 SN74CB3T3245PWR, U2 SN74CB3T3245PWR, U3 SN74CB3T3245PWR, U4 SN74CB3T3245PWR, U5 SN74CB3T3245PWR, U6 TPS3808G33DBVR, U7 TPS3808G50DBVR

Commit message: Simplify carrier to direct bus and slot power; improve schematic readability
Remove bus isolation and USB power circuitry, clarify signal labels, and reflow all schematics onto A4 landscape with larger text. Update PDFs, BOMs, connectivity checks, operating documentation, progress, and remaining tasks.
Parts:
- removed C1, C2, C3, C4, C5, C6, C7: 100nF, symbol A2Ext:C
- removed D2: SS14, symbol A2Ext:D
- removed Q1: 2N7002, Package_TO_SOT_SMD:SOT-23, symbol A2Ext:2N7002
- removed R1: 10k, symbol A2Ext:R
- removed R2: 100k, symbol A2Ext:R
- removed R3: 4.7k, symbol A2Ext:R
- removed U1, U2, U3, U4, U5: SN74CB3T3245PWR, Package_SO:TSSOP-20_4.4x6.5mm_P0.65mm, symbol A2Ext:CB3T3245
- removed U6: TPS3808G33DBVR, Package_TO_SOT_SMD:SOT-23-6, symbol A2Ext:TPS3808
- removed U7: TPS3808G50DBVR, Package_TO_SOT_SMD:SOT-23-6, symbol A2Ext:TPS3808
Connections:
- net GP10 is gone; now on net A8: M1.H1.16 (GPIO10)
- net GP11 is gone; now on net A9: M1.H1.17 (GPIO11)
- net GP12 is gone; now on net A10: M1.H1.18 (GPIO12)
- net GP13 is gone; now on net A11: M1.H1.19 (GPIO13)
- net GP14 is gone; now on net A12: M1.H1.20 (GPIO14)
- net GP15 is gone; now on net A13: M1.H1.21 (GPIO15)
- net GP16 is gone; now on net A14: M1.H1.22 (GPIO16)
- net GP17 is gone; now on net A15: M1.H1.23 (GPIO17)
- net GP18 is gone; now on net D0: M1.H1.24 (GPIO18)
- net GP19 is gone; now on net D1: M1.H1.25 (GPIO19)
- net GP2 is gone; now on net A0: M1.H1.8 (GPIO2)
- net GP20 is gone; now on net D2: M1.H1.26 (GPIO20)
- net GP21 is gone; now on net D3: M1.H1.27 (GPIO21)
- net GP22 is gone; now on net D4: M1.H1.28 (GPIO22)
- net GP23 is gone; now on net D5: M1.H1.29 (GPIO23)
- net GP24 is gone; now on net D6: M1.H1.30 (GPIO24)
- net GP25 is gone; now on net D7: M1.H2.29 (GPIO25)
- net GP26 is gone; now on net RWB: M1.H2.30 (GPIO26)
- net GP27 is gone; now on net DEVSEL_N: M1.H2.27 (GPIO27)
- net GP28 is gone; now on net IOSEL_N: M1.H2.28 (GPIO28)
- net GP29 is gone; now on net IOSTRB_N: M1.H2.25 (GPIO29)
- net GP3 is gone; now on net A1: M1.H1.9 (GPIO3)
- net GP30 is gone; now on net PHI0: M1.H2.26 (GPIO30)
- net GP31 is gone; now on net RES_N: M1.H2.23 (GPIO31)
- net GP32 is gone; now on net IRQ_N: M1.H2.24 (GPIO32)
- net GP33 is gone; now on net NMI_N: M1.H2.21 (GPIO33)
- net GP34 is gone; now on net SYNC: M1.H2.22 (GPIO34)
- net GP4 is gone; now on net A2: M1.H1.10 (GPIO4)
- net GP5 is gone; now on net A3: M1.H1.11 (GPIO5)
- net GP6 is gone; now on net A4: M1.H1.12 (GPIO6)
- net GP7 is gone; now on net A5: M1.H1.13 (GPIO7)
- net GP8 is gone; now on net A6: M1.H1.14 (GPIO8)
- net GP9 is gone; now on net A7: M1.H1.15 (GPIO9)
- net +5V_MOD renamed VSYS
- net A2_A0 renamed A0
- net A2_A1 renamed A1
- net A2_A10 renamed A10
- net A2_A11 renamed A11
- net A2_A12 renamed A12
- net A2_A13 renamed A13
- net A2_A14 renamed A14
- net A2_A15 renamed A15
- net A2_A2 renamed A2
- net A2_A3 renamed A3
- net A2_A4 renamed A4
- net A2_A5 renamed A5
- net A2_A6 renamed A6
- net A2_A7 renamed A7
- net A2_A8 renamed A8
- net A2_A9 renamed A9
- net A2_D0 renamed D0
- net A2_D1 renamed D1
- net A2_D2 renamed D2
- net A2_D3 renamed D3
- net A2_D4 renamed D4
- net A2_D5 renamed D5
- net A2_D6 renamed D6
- net A2_D7 renamed D7
- net A2_DEVSEL_N renamed DEVSEL_N
- net A2_IOSEL_N renamed IOSEL_N
- net A2_IOSTRB_N renamed IOSTRB_N
- net A2_IRQ_N renamed IRQ_N
- net A2_NMI_N renamed NMI_N
- net A2_PHI0 renamed PHI0
- net A2_RES_N renamed RES_N
- net A2_RWB renamed RWB
- net A2_SYNC renamed SYNC
- net GP0 renamed UART_TX
- net GP1 renamed UART_RX
- net GP35 renamed IDC03_GPIO35
- net GP36 renamed IDC04_GPIO36
- net GP37 renamed IDC05_GPIO37
- net GP38 renamed IDC06_GPIO38
- net GP39 renamed IDC07_GPIO39
- net GP40 renamed IDC08_GPIO40
- net GP41 renamed IDC09_GPIO41
- net GP42 renamed IDC10_GPIO42
- net GP43 renamed IDC11_GPIO43
- net GP44 renamed IDC12_GPIO44
- net GP45 renamed IDC13_GPIO45
- net GP46 renamed IDC14_GPIO46
- net GP47 renamed IDC15_GPIO47
- net USB_VBUS: no longer names the net of M1.H1.1 (VBUS (USB))
- no-connect marks 34 -> 14
Other:
- note added: "APPLE II / RP2350B CARRIER Direct bus; slot-only power"
- note added: "MODULE PREPARATION Remove R16, R19, R14, U2. Leave U7/R13/C23 empty. VBUS: NC; USB data only. See carrier README."
- note added: "SIGNAL LABELS _N = active low. UART: carrier TX / RX. H1.n / H2.n: module pins. JP1: open except slot 7. IRQ/NMI: low or release."
- note added: "Slot 25 -> F1/D1 -> VSYS. 5V inputs need powered IOVDD. RUN is separate from /RES. No hot-plugging; flash off-host. Use a 5V fixture at slot 25/26."
- note removed: "BUS ISOLATION / POWER SEQUENCING PROTOTYPE Physical acceptance required before connection to a host."
- note removed: "CB3T devices limit high levels to VCC; not CB3Q substitutes. BUS_OE_N defaults high; Q1 enables only after both supervisors release. Unused channels: NC. Each switch needs a local 100nF capacitor. Slot SYNC jumper is open unless pin 19 is verified."
- note removed: "M1: remove onboard U2; carrier D1/D2 provide explicit supply OR-ing. Remove R16/R19/R14. No secondary flash/PSRAM. IRQ/NMI: firmware assert-low or release only. RUN_N is module reset, separate from Apple II /RES."
- moved on the sheet: C10, C8, C9, D1, F1, F2, J1, J2, JP1, M1, R4

Commit message: Add two-layer prototype PCBs and Gerber packages for all boards
Parts:
- C10, C9: footprint (none) -> A2Ext:C1206
- C8: footprint (none) -> A2Ext:C0805
- D1: footprint (none) -> A2Ext:SS14
- F1, F2: footprint (none) -> A2Ext:PTC1206
- J1: footprint (none) -> A2Ext:AppleII_Edge50
- J2: footprint (none) -> A2Ext:IDC20
- JP1: footprint (none) -> A2Ext:SYNC
- M1: footprint (none) -> A2Ext:WeAct_RP2350B_V1
- R4: footprint (none) -> A2Ext:R0805

Commit message: Revise all prototype PCBs for through-hole assembly
Parts:
- C10, C9: footprint A2Ext:C1206 -> A2Ext:C_Radial_5
- C8: footprint A2Ext:C0805 -> A2Ext:C_Radial_5
- D1: value SS14 -> 1N5819; footprint A2Ext:SS14 -> A2Ext:Schottky_DO41
- F1: footprint A2Ext:PTC1206 -> A2Ext:PTC_MF_R050
- F2: footprint A2Ext:PTC1206 -> A2Ext:PTC_MF_R010
- R4: footprint A2Ext:R0805 -> A2Ext:R_Axial_7.62
